File: CESP.kicad_pcb (KiCad board)
At the start: 2 copper layers, 55.9 x 44.7 mm, 9 parts

Commit message: Somewhat working version, still have some errors
Parts:
- removed LED-1206 (x3): VAL**, LED-1206
- removed SM0603 (x3): Val**, SM0603
- removed SOIC24: VAL**, SOIC24
- removed TSSOP14 (x2): VAL**, TSSOP14
- added C1: C, SM1206, F.Cu at (124.2, 63.5)
- added C2: C, SM0805, F.Cu at (123.7, 90.0)
- added C3: C, SM0603, F.Cu at (122.3, 114.2)
- added C4: C, SM0402, F.Cu at (122.3, 136.9)
- added P1: CONN_1, 1pin, F.Cu at (157.5, 54.9)
- added P10: CONN_1, 1pin, F.Cu at (156.2, 98.6)
- added P11: CONN_1, 1pin, F.Cu at (134.7, 99.4)
- added P12: CONN_1, 1pin, F.Cu at (148.5, 95.2)
- added P13: CONN_1, 1pin, F.Cu at (164.3, 87.1)
- added P14: CONN_1, 1pin, F.Cu at (145.9, 101.7)
- added P15: CONN_1, 1pin, F.Cu at (158.5, 121.8)
- added P16: CONN_1, 1pin, F.Cu at (164.0, 108.2)
- added P17: CONN_1, 1pin, F.Cu at (138.9, 120.1)
- added P18: CONN_1, 1pin, F.Cu at (133.1, 119.9)
- added P19: CONN_1, 1pin, F.Cu at (151.5, 121.7)
- added P2: CONN_1, 1pin, F.Cu at (148.7, 78.9)
- added P20: CONN_1, 1pin, F.Cu at (145.2, 119.9)
- added P21: CONN_1, 1pin, F.Cu at (145.2, 119.8)
- added P22: CONN_1, 1pin, F.Cu at (158.2, 147.2)
- added P23: CONN_1, 1pin, F.Cu at (132.6, 151.6)
- added P24: CONN_1, 1pin, F.Cu at (140.0, 144.0)
- added P25: CONN_1, 1pin, F.Cu at (122.7, 145.7)
- added P26: CONN_1, 1pin, F.Cu at (154.2, 156.0)
- added P27: CONN_1, 1pin, F.Cu at (148.1, 144.1)
- added P28: CONN_1, 1pin, F.Cu at (145.3, 153.0)
- added P3: CONN_1, 1pin, F.Cu at (142.7, 79.2)
- added P4: CONN_1, 1pin, F.Cu at (137.7, 79.2)
- added P5: CONN_1, 1pin, F.Cu at (164.5, 54.7)
- added P6: CONN_1, 1pin, F.Cu at (151.0, 54.6)
- added P7: CONN_1, 1pin, F.Cu at (144.3, 55.5)
- added P8: CONN_1, 1pin, F.Cu at (156.8, 108.7)
- added P9: CONN_1, 1pin, F.Cu at (142.4, 95.4)
- added U1: DS1602, MSOP_8, F.Cu at (144.5, 69.5)
- added U2: DS1602, TSSOP16, F.Cu at (144.8, 87.2)
- added U3: DS1602, SOIC24, F.Cu at (144.5, 109.6)
- added U4: DS1602, SOIC24, F.Cu at (144.3, 130.8)
Other:
- board outline removed
- board text removed: "NOTE: THIS IS JUST A TEST BOARD REMOVE ALL COMPONENTS AND CREATE YOUR OWN INCLUDE SCHEMATIC HOOKUPS/NETLIST"
