File: CESP.sch (KiCad schematic (older format))
At the start: 5 parts

Commit message: Somewhat working version, still have some errors
Parts:
- removed U?: LTC1594CS, TSSOP14, symbol LTC1594CS
- removed U?: TL074, TSSOP14, symbol TL074
- removed U? (x3): TL074, symbol TL074
- added C1, C2, C3, C4: C, ~, symbol C
- added GND1, VCC1: CONNECTOR, ~, symbol CONNECTOR
- added P1, P10, P11, P12, P13, P14, P15, P16, P17, P18, P19, P2, P20, P21, P22, P23, P24, P25, P26, P27, P28, P3, P4, P5, P6, P7, P8, P9: CONN_1, symbol CONN_1
- added U1, U2, U3, U4: DS1602, symbol DS1602
Connections:
- net labels added: GND, GNDPWR, VCC
- wire segments 0 -> 47
Other:
- note removed: "NOTE: THIS IS JUST A TEST BOARD\nREMOVE ALL COMPONENTS AND CREATE YOUR OWN\nINCLUDE SCHEMATIC HOOKUPS/NETLIST"
